File: CANLight.kicad_sch (KiCad schematic)
At the start: 86 parts, among them J1 Screw_Terminal_01x02, J2 Screw_Terminal_01x02, Q1 PNP, Q10 PNP, Q11 PNP, Q12 PNP, Q13 PNP, Q14 PNP, Q15 PNP, Q16 PNP, Q2 PNP, Q3 PNP, Q4 PNP, Q5 PNP, Q6 PNP, Q7 PNP, Q8 PNP, Q9 PNP, U1 MCP23016-I/SP, U2 MIC5504-3.3YM5

Commit message: Initial PCB design
Parts:
- removed C2: 1u, symbol Device:C
- removed U1: MCP23016-I/SP, SPDIP28_300MC_MCH, symbol 2024-03-05_01-39-56:MCP23016-I_SP
- removed U2: MIC5504-3.3YM5, Package_TO_SOT_SMD:SOT-23-5, symbol Regulator_Linear:MIC5504-3.3YM5
- added C3: 22uF, Capacitor_SMD:C_0805_2012Metric, symbol Device:C
- added IC1: TLE42744GS_V33, Library:VREG_TLE42644GHTSA3, symbol TLE42744GS_V33:TLE42744GS_V33
- added R49: 3k3, Resistor_SMD:R_0805_2012Metric, symbol Device:R
- added R50: 1k5, Resistor_SMD:R_0805_2012Metric, symbol Device:R
- added U3: MCP23018-E/SP, Library:SPDIP28_300MC_MCH, symbol 2024-03-05_23-42-54:MCP23018-E_SP
- C1: value 1u -> 22uF; footprint (none) -> Capacitor_SMD:C_0805_2012Metric
- D1, D10, D11, D12, D13, D14, D15, D16, D2, D3, D4, D5, D6, D7, D8, D9: footprint (none) -> Library:HLMP-40XX_BRA
- J1, J2: footprint (none) -> Library:CONN_1935161_PXC
- Q1, Q10, Q11, Q12, Q13, Q14, Q15, Q16, Q2, Q3, Q4, Q5, Q6, Q7, Q8, Q9: footprint (none) -> Library:TO-92-3L_5P33X5P2_ONS
- R1, R10, R11, R12, R13, R14, R15, R16, R17, R18, R19, R2, R20, R21, R22, R23, R24, R25, R26, R27, R28, R29, R3, R30, R31, R32, R33, R34, R35, R36, R37, R38, R39, R4, R40, R41, R42, R43, R44, R45, R46, R47, R48, R5, R6, R7, R8, R9: footprint (none) -> Resistor_SMD:R_0805_2012Metric
Connections:
- net 3V3: now also C3.1, IC1.3 (Q), R49.1, U3.11 (VDD), U3.16 (*RESET)
- net GND: now also C3.2, IC1.2 (GND_1), IC1.4 (GND_2), R50.2, U3.1 (VSS)
- net GP0.0: now also U3.20 (GPA0)
- net GP0.1: now also U3.21 (GPA1)
- net GP0.2: now also U3.22 (GPA2)
- net GP0.3: now also U3.23 (GPA3)
- net GP0.4: now also U3.24 (GPA4)
- net GP0.5: now also U3.25 (GPA5)
- net GP0.6: now also U3.26 (GPA6)
- net GP0.7: now also U3.27 (GPA7)
- net GP1.0: now also U3.3 (GPB0)
- net GP1.1: now also U3.4 (GPB1)
- net GP1.2: now also U3.5 (GPB2)
- net GP1.3: now also R34.1, R35.2, U3.6 (GPB3)
- net GP1.4: now also R37.1, R38.2, U3.7 (GPB4)
- net GP1.5: now also R40.1, R41.2, U3.8 (GPB5)
- net GP1.6: now also R43.1, R44.2, U3.9 (GPB6)
- net GP1.7: now also R46.1, R47.2, U3.10 (GPB7)
- net SCL: now also U3.12 (SCL)
- net SDA: now also U3.13 (SDA)
- net VDD: now also IC1.1 (I)
- new net ADDR: R49.2, R50.1, U3.15 (ADDR)
- no-connect marks 0 -> 6
Other:
- note added: "Addr = 5/16 Vdd Address = 0x22"
- moved on the sheet: C1, D13, D14, D15, D16, Q13, Q14, Q15, Q16, R37, R38, R39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
