File: CANLight.kicad_pcb (KiCad board)
At the start: 2 copper layers, 88 parts, among them IC1 TLE42744GS_V33, J1 Screw_Terminal_01x02, J2 Screw_Terminal_01x02, Q1 PNP, Q10 PNP, Q11 PNP, Q12 PNP, Q13 PNP, Q14 PNP, Q15 PNP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

Commit message: Added Gerbers
Parts:
- moved R50 113.2 mm to (62.8, 86.0), turned to -90 degrees
- moved R49 109.1 mm to (67.0, 85.2), turned to 180 degrees
- moved D9 101.2 mm to (98.0, 96.0), turned to -90 degrees
- moved D16 97.9 mm to (118.0, 156.0), turned to -90 degrees
- moved R48 93.7 mm to (127.0, 160.0), turned to 180 degrees
- moved R26 93.7 mm to (103.5, 94.6), turned to 180 degrees
- moved R46 93.4 mm to (123.5, 157.5), turned to 180 degrees
- moved D12 93.2 mm to (98.0, 156.0), turned to -90 degrees
- moved R25 89.7 mm to (103.5, 98.1), turned to 180 degrees
- moved D10 89.5 mm to (98.0, 116.0), turned to -90 degrees
- moved R47 87.8 mm to (123.5, 154.0), turned to 180 degrees
- moved D11 86.4 mm to (98.0, 136.0), turned to -90 degrees
- moved R34 85.0 mm to (103.5, 158.1), turned to 180 degrees
- moved R35 82.0 mm to (103.5, 154.6), turned to 180 degrees
- moved R36 81.5 mm to (107.0, 160.6), turned to 180 degrees
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Routing:
- net /3V3: track 2.38 -> 354.3 mm
- net /GP1.7: track 4.26 -> 140.6 mm
- net /GP1.6: track 4.26 -> 116.8 mm
- net /GP1.3: track 4.26 -> 114.6 mm
- net /GP0.3: track 4.26 -> 108.5 mm
- net /GP1.2: track 4.26 -> 91.1 mm
- net /GP1.5: track 4.22 -> 88.1 mm
- net /GP0.2: track 4.26 -> 85.1 mm
- net /GP0.7: track 4.26 -> 84.0 mm
- net /GP1.1: track 4.26 -> 72.2 mm
- net /GP0.6: track 4.26 -> 63.2 mm
- net /GP0.1: track 4.26 -> 61.5 mm
- net /GP1.4: track 4.26 -> 59.2 mm
- net /GP0.5: track 4.26 -> 43.3 mm
- net GND: track 8.21 -> 44.5 mm
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- added copper zone on B.Cu, net GND
Other:
- board outline added: 89.2 x 124 mm
- board text added: "I2C CANBUS Status Indicator Designed by Ethan Miller For Team 423"
